Commit message: temporary local commit

File: tecnobody_workbench/urdf/ros2_control/platform_complete_gazebo_robotiq.ros2_control.urdf.xacro (robot description, xacro)
@@ -46,4 +46,12 @@
           <state_interface name="effort" />
         </joint>
+        <transmission name="transmission3">
+          <plugin>transmission_interface/SimpleTransmission</plugin>
+          <actuator name="actuator3" role="actuator3" />
+          <joint name="joint_3" role="joint1">
+            <mechanical_reduction>20.0</mechanical_reduction>
+            <offset>0.0</offset>
+          </joint>
+        </transmission>
       </ros2_control>
       <gazebo>
