Commit message: safe input and z admittance working

File: tecnobody_workbench/urdf/platform_single_actuated.urdf (robot description, URDF)
Before this commit: robot tecnobody, 13 links, 12 joints
Joints:
- joint joint_1: axis 1 0 0 -> (none); limit lower=0 upper=${beam_lenght -4*radius} effort=1000 velocity=2 -> (none); type prismatic -> fixed
- joint joint_3: axis (none) -> 0 0 1; limit (none) -> lower=${-z_height/2} upper=${z_height/2} effort=1000 velocity=2; type fixed -> prismatic
