Commit message: building on tartaglia

File: tecnobody_workbench/urdf/platform_complete_moveit.urdf (robot description, URDF)
Before this commit: robot tecnobody, 13 links, 12 joints
Joints:
- joint joint_1: limit lower=0 upper=3.8 effort=10 velocity=0.5 -> lower=-1.9 upper=1.9 effort=10 velocity=1.0; origin xyz=0.1 -2 1.25 rpy=1.57 0 0 -> xyz=2 -2 1.25 rpy=1.57 0 0
- joint joint_2: limit lower=-1.9 upper=1.9 effort=10 velocity=0.5 -> lower=-1.9 upper=1.9 effort=10 velocity=1.0
- joint joint_3: limit lower=-1 upper=1 effort=10 velocity=0.5 -> lower=-1 upper=1 effort=10 velocity=1.0

Commit message: alignment with np-windows-commented

File: tecnobody_workbench/urdf/platform_complete_moveit.urdf (robot description, URDF)
Before this commit: robot tecnobody, 13 links, 12 joints
Links:
- removed link ee_link
- added link flange_link
- added link link1_beam; visual cylinder length=2 radius=0.1
- link base_link: geometry visual cylinder length=1.5 radius=0.1
- link beam0: geometry visual cylinder length=2 radius=0.1
- link beam1: geometry visual cylinder length=2 radius=0.1
- link beam2: geometry visual cylinder length=2 radius=0.1
- link beam3: geometry visual cylinder length=2 radius=0.1
- link col1: geometry visual cylinder length=1.5 radius=0.1
- link col2: geometry visual cylinder length=1.5 radius=0.1
- link col3: geometry visual cylinder length=1.5 radius=0.1
- link link1: geometry visual box size=0.1 0.1 0.1
- link link3: geometry visual cylinder length=2 radius=0.1
Joints:
- removed joint ee_joint
- removed joint joint_1
- removed joint joint_2
- removed joint joint_3
- added joint flange_joint: type fixed, parent link3, child flange_link, origin xyz=0 0 -0.75 rpy=0 3.141592653589793 -1.5707963267948966
- added joint joint_x: type prismatic, parent link1_beam, child link2, origin xyz=0 0 0 rpy=0 0 0, axis 0 0 1, limit lower=-0.8 upper=0.8 effort=1000 velocity=1
- added joint joint_y: type prismatic, parent base_link, child link1, origin xyz=0 -1 0.75 rpy=-1.5707963267948966 0 3.141592653589793, axis 0 0 -1, limit lower=-1 upper=1 effort=1000 velocity=1
- added joint joint_y_fixed: type fixed, parent link1, child link1_beam, origin xyz=-1 0 0 rpy=0 1.5707963267948966 3.141592653589793
- added joint joint_z: type prismatic, parent link2, child link3, origin xyz=0 0 0 rpy=-1.5707963267948966 0 0, axis 0 0 1, limit lower=-0.5 upper=0.2 effort=1000 velocity=1
- joint base2world: origin xyz=0 0 0 rpy=0 0 -1.57 -> xyz=0 0 0 rpy=0 0 -1.5707963267948966
- joint beam0_joint: origin xyz=0 -2 1.25 rpy=1.57 0 0 -> xyz=0 -1 0.75 rpy=1.5707963267948966 0 0
- joint beam1_joint: origin xyz=-2 0 1.25 rpy=0 1.57 0 -> xyz=-1 0 0.75 rpy=0 1.5707963267948966 0
- joint beam2_joint: origin xyz=0 -2 1.25 rpy=1.57 0 0 -> xyz=0 -1 0.75 rpy=1.5707963267948966 0 0
- joint beam3_joint: origin xyz=2 0 1.25 rpy=0 1.57 0 -> xyz=1 0 0.75 rpy=0 1.5707963267948966 0
- joint col1_joint: origin xyz=-4 0 0 rpy=0 0 1.57 -> xyz=-2 0 0 rpy=0 0 1.5707963267948966
- joint col2_joint: origin xyz=-4 -4 0 rpy=0 0 1.57 -> xyz=-2 -2 0 rpy=0 0 1.5707963267948966
- joint col3_joint: origin xyz=0 -4 0 rpy=0 0 1.57 -> xyz=0 -2 0 rpy=0 0 1.5707963267948966
