Commit message: three motor working and calibrated

File: tecnobody_workbench/urdf/platform_complete.urdf (robot description, URDF)
Before this commit: robot tecnobody, 13 links, 12 joints
Joints:
- joint joint_1: axis 1 0 0 -> 0 0 1; child link1 -> link2; limit lower=0 upper=${beam_lenght -4*radius} effort=1000 velocity=2 -> lower=${-beam_lenght/2+2*radius} upper=${beam_lenght/2-2*radius} effort=1000 velocity=2; origin xyz=0.1 ${-beam_lenght/2} ${col_height/2} rpy=1.57 0 0 -> xyz=0 0 0 rpy=0 0 0; parent base_link -> link1
- joint joint_2: axis 0 0 1 -> 1 0 0; child link2 -> link1; limit lower=${-beam_lenght/2+2*radius} upper=${beam_lenght/2-2*radius} effort=1000 velocity=2 -> lower=0 upper=${beam_lenght -4*radius} effort=1000 velocity=2; origin xyz=0 0 0 rpy=0 0 0 -> xyz=0.1 ${-beam_lenght/2} ${col_height/2} rpy=1.57 0 0; parent link1 -> base_link

Commit message: alignment

File: tecnobody_workbench/urdf/platform_complete.urdf (robot description, URDF)
Before this commit: robot tecnobody, 13 links, 12 joints
Links:
- added link link1_beam; visual cylinder length=${beam_lenght} radius=${radius}
- link link1: geometry visual box size=0.1 0.1 0.1
Joints:
- removed joint joint_1
- removed joint joint_2
- removed joint joint_3
- added joint joint_x: type prismatic, parent link1_beam, child link2, origin xyz=0 0 0 rpy=0 0 0, axis 0 0 1, limit lower=${-beam_lenght/2+2*radius} upper=${beam_lenght/2-2*radius} effort=1000 velocity=1
- added joint joint_y: type prismatic, parent base_link, child link1, origin xyz=0 ${-beam_lenght/2} ${col_height/2} rpy=-1.57 0 0, axis 0 0 1, limit lower=${-beam_lenght/2+2*radius} upper=${beam_lenght/2-2*radius} effort=1000 velocity=1
- added joint joint_y_fixed: type fixed, parent link1, child link1_beam, origin xyz=${beam_lenght/2} 0 0 rpy=0 1.57 0
- added joint joint_z: type prismatic, parent link2, child link3, origin xyz=0 0 0 rpy=1.57 0 0, axis 0 0 1, limit lower=${-z_height/2} upper=${z_height/2} effort=1000 velocity=1
- joint ee_joint: origin xyz=0 0 ${-z_height/2} rpy=0 3.14 0 -> xyz=0 0 ${-z_height/2} rpy=0 3.14 -1.57

Commit message: minor fixes

File: tecnobody_workbench/urdf/platform_complete.urdf (robot description, URDF)
Before this commit: robot tecnobody, 14 links, 13 joints
Links:
- added link flange_link
- added link ft_link
Joints:
- added joint flange_joint: type fixed, parent link3, child flange_link, origin xyz=0 0 ${-z_height/2} rpy=0 ${PI} ${-PI/2.0}
- added joint joint_yaw: type revolute, parent flange_link, child ft_link, origin xyz=0 0 0.04 rpy=0 0 ${PI}, axis 0 0 1, limit lower=-${PI} upper=${PI} effort=1000 velocity=1
- joint base2world: origin xyz=0 0 0 rpy=0 0 -1.57 -> xyz=0 0 0 rpy=0 0 ${-PI/2.0}
- joint beam0_joint: origin xyz=0 ${-beam_lenght/2} ${col_height/2} rpy=1.57 0 0 -> xyz=0 ${-beam_lenght/2} ${col_height/2} rpy=${PI/2.0} 0 0
- joint beam1_joint: origin xyz=${-beam_lenght/2} 0 ${col_height/2} rpy=0 1.57 0 -> xyz=${-beam_lenght/2} 0 ${col_height/2} rpy=0 ${PI/2.0} 0
- joint beam2_joint: origin xyz=0 ${-beam_lenght/2} ${col_height/2} rpy=1.57 0 0 -> xyz=0 ${-beam_lenght/2} ${col_height/2} rpy=${PI/2.0} 0 0
- joint beam3_joint: origin xyz=${beam_lenght/2} 0 ${col_height/2} rpy=0 1.57 0 -> xyz=${beam_lenght/2} 0 ${col_height/2} rpy=0 ${PI/2.0} 0
- joint col1_joint: origin xyz=${-beam_lenght} 0 0 rpy=0 0 1.57 -> xyz=${-beam_lenght} 0 0 rpy=0 0 ${PI/2.0}
- joint col2_joint: origin xyz=${-beam_lenght} ${-beam_lenght} 0 rpy=0 0 1.57 -> xyz=${-beam_lenght} ${-beam_lenght} 0 rpy=0 0 ${PI/2.0}
- joint col3_joint: origin xyz=0 ${-beam_lenght} 0 rpy=0 0 1.57 -> xyz=0 ${-beam_lenght} 0 rpy=0 0 ${PI/2.0}
- joint ee_joint: origin xyz=0 0 ${-z_height/2} rpy=0 3.14 -1.57 -> xyz=0 0 0.07 rpy=0 0 0; parent link3 -> ft_link
- joint joint_y: axis 0 0 1 -> 0 0 -1; origin xyz=0 ${-beam_lenght/2} ${col_height/2} rpy=-1.57 0 0 -> xyz=0 ${-beam_lenght/2} ${col_height/2} rpy=${-PI/2.0} 0 ${PI}
- joint joint_y_fixed: origin xyz=${beam_lenght/2} 0 0 rpy=0 1.57 0 -> xyz=-${beam_lenght/2} 0 0 rpy=0 ${PI/2.0} ${PI}
- joint joint_z: origin xyz=0 0 0 rpy=1.57 0 0 -> xyz=0 0 0 rpy=-${PI/2.0} 0 0

Commit message: minor fixes

File: tecnobody_workbench/urdf/platform_complete.urdf (robot description, URDF)
Before this commit: robot tecnobody, 16 links, 15 joints
Joints:
- joint joint_x: limit lower=${-beam_lenght/2+2*radius} upper=${beam_lenght/2-2*radius} effort=1000 velocity=1 -> lower=${-beam_lenght/2+2*radius} upper=${beam_lenght/2-2*radius} effort=1000 velocity=7.0
- joint joint_y: limit lower=${-beam_lenght/2+2*radius} upper=${beam_lenght/2-2*radius} effort=1000 velocity=1 -> lower=${-beam_lenght/2+2*radius} upper=${beam_lenght/2-2*radius} effort=1000 velocity=7.0
- joint joint_yaw: limit lower=-${PI} upper=${PI} effort=1000 velocity=1 -> lower=-${PI} upper=${PI} effort=1000 velocity=7.0
- joint joint_z: limit lower=${-z_height/2} upper=${z_height/2} effort=1000 velocity=1 -> lower=${-z_height/2} upper=${z_height/2} effort=1000 velocity=7.0
